File: drv8424epwpr_carrier/drv8424epwpr_carrier.kicad_pcb (KiCad board)
At the start: 2 copper layers, 27 parts, among them J1 Input_01x08, J2 Output_01x08, J3 POW_01x02, U1 DRV8424EPWPR, U2 DMP4013LFG-7

Commit message: update layout
Parts:
- moved LED1 35.7 mm to (103.8, 61.5)
- moved LED3 35.7 mm to (103.8, 64.3)
- moved LED5 35.7 mm to (103.8, 67.1)
- moved CR1 33.9 mm to (113.9, 56.8)
- moved U1 30.2 mm to (64.4, 66.3)
- moved R1 25.9 mm to (88.4, 45.0)
- moved R1_REFA1 25.9 mm to (88.4, 58.0)
- moved R1_REFB1 25.9 mm to (88.4, 61.3)
- moved R2 25.9 mm to (88.4, 48.3)
- moved R2_REFA1 25.9 mm to (88.4, 64.6)
- moved R2_REFB1 25.9 mm to (88.4, 67.8)
- moved R3 25.9 mm to (88.4, 51.5)
- moved R4 25.9 mm to (88.4, 54.8)
- moved R_nFAULT1 25.9 mm to (88.4, 71.1)
- moved J2 23.5 mm to (52.5, 58.8)
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Connections:
- J1 pad 1: +3V3 -> NSLEEP
- J1 pad 2: GND -> AEN
- J1 pad 3: NFAULT -> APH
- J1 pad 4: NSLEEP -> BEN
- J1 pad 5: AEN -> BPH
- J1 pad 6: APH -> NFAULT
- J1 pad 7: BEN -> GND
- J1 pad 8: BPH -> +3V3
- J2 pad 7: BOUT2 -> BOUT1
- J2 pad 8: BOUT1 -> BOUT2
Other:
- board outline added: 28 x 36 mm

Commit message: update layout
Parts:
- LED1: value YELLOW -> YLW
- LED2, LED4: value GREEN -> GRN
- moved CR1 58.0 mm to (59.5, 77.0), turned to -90 degrees
- moved LED2 53.7 mm to (51.5, 53.5), turned to 90 degrees
- moved LED5 52.6 mm to (53.5, 82.5), turned to 90 degrees
- moved LED4 52.0 mm to (51.5, 82.5), turned to -90 degrees
- moved C_VCP 51.7 mm to (57.5, 68.6), turned to -90 degrees
- moved LED3 51.4 mm to (53.5, 53.5), turned to -90 degrees
- moved R1 44.5 mm to (56.0, 75.6), turned to 90 degrees
- moved R3 44.1 mm to (56.0, 81.5), turned to -90 degrees
- moved LED1 40.5 mm to (70.5, 84.5), turned to 180 degrees
- moved C_SW 39.0 mm to (70.6, 62.5)
- moved R2 33.5 mm to (56.0, 57.1), turned to 90 degrees
- moved R4 32.5 mm to (70.6, 82.0), turned to 180 degrees
- moved U2 31.3 mm to (63.9, 77.0)
- moved C_DV 28.4 mm to (65.6, 73.5), turned to 180 degrees
- moved REFB1 22.0 mm to (69.5, 72.6), turned to 90 degrees
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- renumbered C_DVDD1 to C_DV, C_SW1 to C_SW, C_VCP1 to C_VCP, R1_REFA1 to REFA1, R2_REFA1 to REFA2, R1_REFB1 to REFB1, R2_REFB1 to REFB2, R_nFAULT1 to R_nF

Commit message: start routing
Parts:
- added G***: LOGO, model_lib:bearhead, F.Cu at (75.0, 54.5)
- moved U2 1.50 mm to (62.4, 77.0)
- moved CR1 1.00 mm to (58.5, 77.0)
- moved LED2 1.00 mm to (51.5, 54.5)
- moved LED3 1.00 mm to (53.5, 54.5)
- moved R2 1.00 mm to (56.0, 58.1)
Routing:
- net VM: track 0.00 -> 13.8 mm
- net VIN: track 0.00 -> 8.93 mm
- net Net-(U1-CPL): track 0.00 -> 6.59 mm
- net Net-(U1-CPH): track 0.00 -> 2.65 mm

Commit message: update layout
Routing:
- net VREFA: track 0.00 -> 24.5 mm, vias 0 -> 1
- net VM: track 13.8 -> 37.7 mm, vias 0 -> 2
- net AOUT2: track 0.00 -> 23.1 mm
- net NFAULT: track 0.00 -> 18.6 mm
- net AOUT1: track 0.00 -> 15.6 mm
- net DVDD: track 0.00 -> 9.90 mm, vias 0 -> 2
- net Net-(LED2-Pad2): track 0.00 -> 6.40 mm
- net VREFB: track 0.00 -> 6.10 mm
- net Net-(U2-G): track 0.00 -> 5.81 mm
- net +3V3: track 0.00 -> 3.53 mm

Commit message: update layout
Parts:
- removed CR1: 15V, MMSZ5245B_7_F:SOD123_DIO
- moved G*** 29.0 mm to (70.0, 83.1)
- moved LED1 11.9 mm to (60.6, 77.9), turned to 90 degrees
- moved REFA1 10.1 mm to (65.7, 76.5), turned to 180 degrees
- moved REFA2 9.46 mm to (65.7, 74.2), turned to 0 degrees
- moved R_nF 8.16 mm to (70.5, 69.3)
- moved C_VM4 7.58 mm to (68.5, 56.7), turned to 90 degrees
- moved C_VM3 7.44 mm to (61.1, 56.7), turned to 90 degrees
- moved C_VM2 7.14 mm to (58.0, 70.2), turned to 90 degrees
- moved R4 5.80 mm to (65.7, 78.9)
- moved REFB2 5.32 mm to (70.4, 77.7), turned to 0 degrees
- moved C_DV 5.29 mm to (70.5, 71.7), turned to 0 degrees
- moved U2 4.93 mm to (57.5, 77.2), turned to -90 degrees
- moved C_VCP 4.44 mm to (55.6, 64.6)
- moved REFB1 2.90 mm to (70.4, 75.4), turned to 180 degrees
- moved R1 2.78 mm to (57.9, 73.6), turned to 0 degrees
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Routing:
- net VM: track 37.7 -> 0.00 mm, vias 2 -> 0
- net VREFA: track 24.5 -> 0.00 mm, vias 1 -> 0
- net AOUT2: track 23.1 -> 0.00 mm
- net NFAULT: track 18.6 -> 0.00 mm
- net AOUT1: track 15.6 -> 0.00 mm
- net NSLEEP: track 0.00 -> 11.7 mm
- net BPH: track 0.00 -> 9.93 mm
- net DVDD: track 9.90 -> 0.00 mm, vias 2 -> 0
- net AEN: track 0.00 -> 9.80 mm
- net BEN: track 0.00 -> 9.15 mm
- net APH: track 0.00 -> 9.01 mm
- net VIN: track 8.93 -> 0.00 mm
- net Net-(U1-CPL): track 6.59 -> 0.00 mm
- net Net-(LED2-Pad2): track 6.40 -> 0.00 mm
- net VREFB: track 6.10 -> 0.00 mm
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Other:
- board size 28 x 36 mm -> 26.5 x 35.4 mm

Commit message: update layout
Parts:
- moved C_VCP 3.40 mm to (55.7, 61.2)
- moved LED1 1.62 mm to (61.7, 76.7)
- moved C_VM1 0.77 mm to (58.1, 63.8)
- moved LED4 0.50 mm to (51.9, 81.5)
- moved R3 0.50 mm to (56.0, 82.3)
- moved LED5 0.50 mm to (53.8, 81.7)
Routing:
- net DVDD: track 0.00 -> 13.1 mm, vias 0 -> 2
- net VREFB: track 0.00 -> 11.0 mm
- net VIN: track 0.00 -> 10.6 mm
- net +3V3: track 0.00 -> 9.78 mm
- net VREFA: track 0.00 -> 8.42 mm, vias 0 -> 2
- net NFAULT: track 0.00 -> 3.14 mm

Commit message: update pcb
Parts:
- added CR1: 15V, MMSZ5245B_7_F:SOD123_DIO, F.Cu at (86.0, 65.1)
- added C_DVDD1: 1uF, Capacitor_SMD:C_0805_2012Metric, F.Cu at (80.7, 65.1)
- added C_SW1: 0.022uF, Capacitor_SMD:C_0805_2012Metric, F.Cu at (80.7, 68.1)
- added C_VCP1: 0.22uF, Capacitor_SMD:C_0805_2012Metric, F.Cu at (80.7, 71.1)
- C_VM1, C_VM2: footprint C0805C103K8RACTU:CAPC220145_88N_KEM -> Capacitor_SMD:C_0805_2012Metric
- LED1: value YLW -> YELLOW; footprint APHCM2012SYCK_F01:LED_APHCM2012SYCK-F01 -> LED_SMD:LED_0805_2012Metric
- LED2, LED4: value GRN -> GREEN; footprint APHCM2012CGCK_F01:LED_APHCM2012CGCK-F01_KNB -> LED_SMD:LED_0805_2012Metric
- LED3, LED5: footprint APHCM2012SURCK_F01:LED_APHCM2012SURCK-F01 -> LED_SMD:LED_0805_2012Metric
- R1: footprint RC1206FR_07100KL:RC1206N_YAG -> Resistor_SMD:R_1206_3216Metric
- R1_REFA1: renamed from REFA1; footprint RC1206FR_0747KL:RC1206N_YAG -> Resistor_SMD:R_1206_3216Metric
- R1_REFB1: renamed from REFB1; footprint RC1206FR_0747KL:RC1206N_YAG -> Resistor_SMD:R_1206_3216Metric
- R2, R3, R4: footprint RC1206FR_07590RL:RC1206N_YAG -> Resistor_SMD:R_1206_3216Metric
- R2_REFA1: renamed from REFA2; footprint RC1206FR_0716KL:RC1206N_YAG -> Resistor_SMD:R_1206_3216Metric
- R2_REFB1: renamed from REFB2; footprint RC1206FR_0716KL:RC1206N_YAG -> Resistor_SMD:R_1206_3216Metric
- R_nFAULT1: renamed from R_nF; footprint RC1206FR_0710KL:RC1206N_YAG -> Resistor_SMD:R_1206_3216Metric

Commit message: update layout
Parts:
- removed C_DV: 1uF, GRM319R71A105KA01D:CAPC3216X95N
- removed the C_SW at (70.5, 63.0)
- removed C_VCP: 0.22uF, C1206C224K4RACTU:CAPC340180_100N_KEM
- removed LED5: RED, LED_SMD:LED_0805_2012Metric
- moved CR1 41.3 mm to (45.7, 74.1)
- moved C_VCP1 26.5 mm to (55.8, 61.9), turned to 90 degrees
- moved C_DVDD 12.8 mm to (70.4, 72.6)
- moved C_SW 11.7 mm to (70.0, 63.2)
- moved R2 2.15 mm to (56.4, 53.3)
- moved R3 2.03 mm to (58.0, 82.1)
- renumbered C_DVDD1 to C_DVDD, C_SW1 to C_SW
Routing:
- net DVDD: track 13.1 -> 0.00 mm, vias 2 -> 0
- net NSLEEP: track 11.7 -> 0.00 mm
- net VREFB: track 11.0 -> 0.00 mm
- net VIN: track 10.6 -> 0.00 mm
- net BPH: track 9.93 -> 0.00 mm
- net AEN: track 9.80 -> 0.00 mm
- net +3V3: track 9.78 -> 0.00 mm
- net BEN: track 9.15 -> 0.00 mm
- net APH: track 9.01 -> 0.00 mm
- net VREFA: track 8.42 -> 0.00 mm, vias 2 -> 0
- net NFAULT: track 3.14 -> 0.00 mm
