File: drv8424epwpr_carrier/drv8424epwpr_carrier.kicad_pcb (KiCad board)
At the start: 2 copper layers, 26.5 x 35.4 mm, 27 parts, among them J1 Input_01x08, J2 Output_01x08, J3 POW_01x02, U1 DRV8424EPWPR, U2 DMP4013LFG-7

Commit message: update layout
Parts:
- added LED5: RED, LED_SMD:LED_0805_2012Metric, F.Cu at (54.0, 82.1)
- moved G*** 12.2 mm to (82.1, 81.8)
- moved CR1 11.8 mm to (57.5, 73.8), turned to 180 degrees
- moved R4 8.03 mm to (58.6, 82.7), turned to -90 degrees
- moved R1 4.12 mm to (55.7, 70.1), turned to 90 degrees
- moved R_nFAULT 3.06 mm to (72.0, 72.0), turned to 90 degrees
- moved R1_REFA 2.16 mm to (65.9, 78.7)
- moved R2 2.08 mm to (56.3, 55.4)
- moved R2_REFB 2.07 mm to (71.0, 79.7)
- moved R3 1.86 mm to (56.2, 82.7)
- moved R2_REFA 1.56 mm to (65.9, 75.7)
- moved R1_REFB 1.43 mm to (71.0, 76.7)
- moved C_DVDD 1.19 mm to (69.2, 72.6), turned to -90 degrees
- moved U2 0.69 mm to (56.8, 77.3)
- moved LED4 0.68 mm to (51.9, 82.2)
- moved LED3 0.64 mm to (54.1, 56.0)
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- renumbered C_SW to C_SW1, R1_REFA1 to R1_REFA, R1_REFB1 to R1_REFB, R2_REFA1 to R2_REFA, R2_REFB1 to R2_REFB, R_nFAULT1 to R_nFAULT

Commit message: update layout
Parts:
- moved R1 3.73 mm to (57.0, 73.6), turned to 0 degrees
- moved CR1 3.71 mm to (60.4, 76.0), turned to -90 degrees
- moved LED1 0.92 mm to (62.5, 76.7), turned to 90 degrees

Commit message: update routing
Parts:
- moved G*** 18.9 mm to (70.8, 66.8)
- moved U2 6.96 mm to (63.5, 75.5), turned to 0 degrees
- moved R2_REFA1 5.87 mm to (70.8, 79.0)
- moved R1_REFA1 5.36 mm to (70.8, 76.5)
- moved R1_REFB1 4.91 mm to (70.0, 81.5)
- moved R2_REFB1 4.45 mm to (70.0, 84.0)
- moved C_DVDD1 2.95 mm to (67.2, 74.8)
- moved R1 2.73 mm to (57.5, 76.3), turned to 90 degrees
- moved LED1 2.29 mm to (62.5, 79.0), turned to 0 degrees
- moved R_nFAULT1 1.78 mm to (71.0, 73.5), turned to 180 degrees
- moved C_VM2 1.68 mm to (58.1, 71.8), turned to -90 degrees
- moved C_VM1 1.00 mm to (58.1, 62.9), turned to 90 degrees
- moved CR1 0.77 mm to (59.8, 75.6)
- moved C_VM3 0.63 mm to (61.5, 56.1)
- moved C_VM4 0.63 mm to (68.9, 56.1)
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- renumbered C_DVDD to C_DVDD1, R1_REFA to R1_REFA1, R1_REFB to R1_REFB1, R2_REFA to R2_REFA1, R2_REFB to R2_REFB1, R_nFAULT to R_nFAULT1
Connections:
- J2 pad 1: AOUT1 -> VM
- J2 pad 2: AOUT2 -> GND
- J2 pad 3: VREFA -> AOUT1
- J2 pad 4: VM -> AOUT2
- J2 pad 5: GND -> BOUT1
- J2 pad 6: VREFB -> BOUT2
- J2 pad 7: BOUT1 -> VREFA
- J2 pad 8: BOUT2 -> VREFB
Routing:
- net VM: track 0.00 -> 37.0 mm
- net AOUT2: track 0.00 -> 27.0 mm, vias 0 -> 2
- net BOUT1: track 0.00 -> 23.3 mm, vias 0 -> 2
- net BOUT2: track 0.00 -> 21.2 mm
- net AOUT1: track 0.00 -> 18.1 mm, vias 0 -> 2
- net VREFB: track 0.00 -> 15.7 mm, vias 0 -> 2
- net DVDD: track 0.00 -> 14.4 mm
- net VREFA: track 0.00 -> 13.5 mm, vias 0 -> 2
- net NFAULT: track 0.00 -> 11.2 mm
- net NSLEEP: track 0.00 -> 11.1 mm
- net BPH: track 0.00 -> 9.93 mm
- net AEN: track 0.00 -> 9.80 mm
- net BEN: track 0.00 -> 9.15 mm
- net APH: track 0.00 -> 9.01 mm
- net VIN: track 0.00 -> 7.52 mm
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
Commit message: update routing
Parts:
- moved G*** 1.67 mm to (71.0, 68.4)
Routing:
- net VREFA: track 13.5 -> 36.7 mm, vias 2 -> 4
- net VREFB: track 15.7 -> 32.8 mm, vias 2 -> 3
- net Net-(U2-G): track 0.00 -> 6.68 mm, vias 0 -> 2
- net VM: track 37.0 -> 39.5 mm
Changed lines of the file:
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@@
 	(footprint "model_lib:bearhead"
 		(layer "F.Cu")
-		(at 70.75 66.75)
+		(at 71 68.4)
 		(property "Reference" "G***"
 			(at -0.127 2.9718 0)
@@
 	)
 	(segment
+		(start 60.5409 70.982586)
+		(end 58.146986 70.982586)
+		(width 0.5)
+		(layer "F.Cu")
+		(net 1)
+	)
+	(segment
 		(start 59.75 72.5856)
 		(end 58.0644 70.9)
@@
 	)
 	(segment
+		(start 58.146986 70.982586)
+		(end 58.0644 70.9)
+		(width 0.5)
+		(layer "F.Cu")
+		(net 1)
+	)
+	(segment
 		(start 61.2748 73.875)
 		(end 61.8998 74.5)
@@
 	)
 	(segment
+		(start 57.925 77.325)
+		(end 57.5 77.75)
+		(width 0.2)
+		(layer "F.Cu")
+		(net 2)
+	)
+	(segment
+		(start 59.75 77.325)
+		(end 57.925 77.325)
+		(width 0.2)
+		(layer "F.Cu")
+		(net 2)
+	)
+	(segment
+		(start 60.732038 77.735241)
+		(end 60.160241 77.735241)
+		(width 0.2)
+		(layer "F.Cu")
+		(net 2)
+	)
+	(segment
+		(start 60.160241 77.735241)
+		(end 59.75 77.325)
+		(width 0.2)
+		(layer "F.Cu")
+		(net 2)
+	)
+	(segment
+		(start 61.8998 76.449998)
+		(end 62.249998 76.449998)
+		(width 0.2)
+		(layer "F.Cu")
+		(net 2)
+	)
+	(segment
+		(start 62.249998 76.449998)
+		(end 62.6 76.8)
+		(width 0.2)
+		(layer "F.Cu")
+		(net 2)
+	)
+	(via
+		(at 62.6 76.8)
+		(size 0.6)
+		(drill 0.3)
+		(layers "F.Cu" "B.Cu")
+		(net 2)
+	)
+	(via
+		(at 60.732038 77.735241)
+		(size 0.6)
+		(drill 0.3)
+		(layers "F.Cu" "B.Cu")
+		(net 2)
+	)
+	(segment
+		(start 62.4 77)
+		(end 61.467279 77)
+		(width 0.2)
+		(layer "B.Cu")
+		(net 2)
+	)
+	(segment
+		(start 62.6 76.8)
+		(end 62.4 77)
+		(width 0.2)
+		(layer "B.Cu")
+		(net 2)
+	)
+	(segment
+		(start 61.467279 77)
+		(end 60.732038 77.735241)
+		(width 0.2)
+		(layer "B.Cu")
+		(net 2)
+	)
+	(segment
 		(start 72.25 76.5)
 		(end 70.425 74.675)
@@
 		(net 18)
 	)
+	(segment
+		(start 52.5 78.9)
+		(end 52.8 79.2)
+		(width 0.2)
+		(layer "F.Cu")
+		(net 18)
+	)
+	(segment
+		(start 52.5 77.7)
+		(end 52.5 78.9)
+		(width 0.2)
+		(layer "F.Cu")
+		(net 18)
+	)
 	(via
 		(at 68.388978 70.866985)
@@
 		(net 18)
 	)
+	(via
+		(at 52.8 79.2)
+		(size 0.6)
+		(drill 0.3)
+		(layers "F.Cu" "B.Cu")
+		(net 18)
+	)
 	(segment
 		(start 68.388978 70.866985)
@@
 	)
 	(segment
+		(start 52.8 79.2)
+		(end 66.55 79.2)
+		(width 0.2)
+		(layer "B.Cu")
+		(net 18)
+	)
+	(segment
+		(start 66.55 79.2)
+		(end 67.75 78)
+		(width 0.2)
+		(layer "B.Cu")
+		(net 18)
+	)
+	(segment
 		(start 68.388978 77.361022)
 		(end 67.75 78)
@@
 	)
 	(segment
+		(start 51.35 79.3278)
+		(end 51.4222 79.4)
+		(width 0.2)
+		(layer "F.Cu")
+		(net 20)
+	)
+	(segment
+		(start 52.5 75.16)
+		(end 51.35 76.31)
+		(width 0.2)
+		(layer "F.Cu")
+		(net 20)
+	)
+	(segment
 		(start 69.325 79)
 		(end 69.325 76.5)
@@
 	)
 	(segment
+		(start 51.35 76.31)
+		(end 51.35 79.3278)
+		(width 0.2)
+		(layer "F.Cu")
+		(net 20)
+	)
+	(segment
 		(start 69.825 76)
 		(end 69.325 76.5)
@@
 	)
 	(segment
+		(start 68.525 79.8)
+		(end 69.325 79)
+		(width 0.2)
+		(layer "F.Cu")
+		(net 20)
+	)
+	(segment
 		(start 70.75 76)
 		(end 69.825 76)
@@
 		(net 20)
 	)
+	(segment
+		(start 68.35 79.8)
+		(end 68.525 79.8)
+		(width 0.2)
+		(layer "F.Cu")
+		(net 20)
+	)
 	(via
 		(at 70.75 76)
@@
 	)
 	(via
+		(at 51.4222 79.4)
+		(size 0.6)
+		(drill 0.3)
+		(layers "F.Cu" "B.Cu")
+		(net 20)
+	)
+	(via
+		(at 68.35 79.8)
+		(size 0.6)
+		(drill 0.3)
+		(layers "F.Cu" "B.Cu")
+		(net 20)
+	)
+	(via
 		(at 69.07479 70.45508)
 		(size 0.6)
@@
 		(width 0.2)
 		(layer "B.Cu")
+		(net 20)
+	)
+	(segment
+		(start 51.4222 79.4)
+		(end 51.8222 79.8)
+		(width 0.2)
+		(layer "B.Cu")
+		(net 20)
+	)
+	(segment
+		(start 51.8222 79.8)
+		(end 68.35 79.8)
+		(width 0.2)
+		(layer "B.Cu")

Commit message: update routing
Parts:
- moved CR1 1.29 mm to (58.8, 76.5)
- moved U2 0.91 mm to (62.6, 75.6)
- moved R1 0.90 mm to (56.6, 76.3)
- renumbered C_DVDD1 to C_DV
Routing:
- net GND: track 0.00 -> 119.4 mm, vias 0 -> 2
- net VM: track 39.5 -> 54.7 mm, vias 0 -> 4
- net VIN: track 7.52 -> 11.6 mm
- net Net-(U2-G): track 6.68 -> 5.70 mm, vias 2 -> 0
- net BOUT1: track 23.3 -> 22.3 mm, vias 2 -> 1
- net AOUT2: track 27.0 -> 26.4 mm
- net AOUT1: track 18.1 -> 18.5 mm, vias 2 -> 1
